File: pcb/nixie_clock/Nixie_Block.kicad_pcb (KiCad board)
At the start: 6 copper layers, 25 parts, among them U1 MSD42WT1G, U10 MSD42WT1G, U11 MSD42WT1G, U12 MSD42WT1G, U2 MSD42WT1G, U3 MSD42WT1G, U4 MSD42WT1G, U5 MSD42WT1G, U6 MSD42WT1G, U7 MSD42WT1G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

Commit message: fixing some issues.
Changed lines of the file:
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@@
 			(layer "B.CrtYd")
+		)
+		(fp_text user "2"
+			(at -7.941671 0.964293 -83.076)
+			(unlocked yes)
+			(layer "B.SilkS")
+			(effects
+				(font
+					(size 1 1)
+					(thickness 0.1)
+				)
+				(justify bottom mirror)
+			)
+		)
+		(fp_text user "5"
+			(at -1.914525 -7.767535 -166.153)
+			(unlocked yes)
+			(layer "B.SilkS")
+			(effects
+				(font
+					(size 1 1)
+					(thickness 0.1)
+				)
+				(justify bottom mirror)
+			)
+		)
+		(fp_text user "1"
+			(at -6.583871 4.544518 -55.384)
+			(unlocked yes)
+			(layer "B.SilkS")
+			(effects
+				(font
+					(size 1 1)
+					(thickness 0.1)
+				)
+				(justify bottom mirror)
+			)
+		)
+		(fp_text user "6"
+			(at 1.914525 -7.767535 166.153)
+			(unlocked yes)
+			(layer "B.SilkS")
+			(effects
+				(font
+					(size 1 1)
+					(thickness 0.1)
+				)
+				(justify bottom mirror)
+			)
+		)
+		(fp_text user "0"
+			(at 6.583871 4.544518 55.384)
+			(unlocked yes)
+			(layer "B.SilkS")
+			(effects
+				(font
+					(size 1 1)
+					(thickness 0.1)
+				)
+				(justify bottom mirror)
+			)
+		)
+		(fp_text user "4"
+			(at -5.304981 -5.988086 -138.461)
+			(unlocked yes)
+			(layer "B.SilkS")
+			(effects
+				(font
+					(size 1 1)
+					(thickness 0.1)
+				)
+				(justify bottom mirror)
+			)
+		)
+		(fp_text user "3"
+			(at -7.48013 -2.836839 -110.769)
+			(unlocked yes)
+			(layer "B.SilkS")
+			(effects
+				(font
+					(size 1 1)
+					(thickness 0.1)
+				)
+				(justify bottom mirror)
+			)
+		)
+		(fp_text user "CR"
+			(at 3.717785 7.083648 27.692)
+			(unlocked yes)
+			(layer "B.SilkS")
+			(effects
+				(font
+					(size 1 1)
+					(thickness 0.1)
+				)
+				(justify bottom mirror)
+			)
+		)
+		(fp_text user "8"
+			(at 7.48013 -2.836839 110.769)
+			(unlocked yes)
+			(layer "B.SilkS")
+			(effects
+				(font
+					(size 1 1)
+					(thickness 0.1)
+				)
+				(justify bottom mirror)
+			)
+		)
+		(fp_text user "CL"
+			(at -3.717785 7.083648 -27.692)
+			(unlocked yes)
+			(layer "B.SilkS")
+			(effects
+				(font
+					(size 1 1)
+					(thickness 0.1)
+				)
+				(justify bottom mirror)
+			)
+		)
+		(fp_text user "A"
+			(at 0 8 0)
+			(unlocked yes)
+			(layer "B.SilkS")
+			(effects
+				(font
+					(size 1 1)
+					(thickness 0.1)
+				)
+				(justify bottom mirror)
+			)
 		)
 		(fp_text user "9"
@@
 			)
 		)
-		(fp_text user "CR"
-			(at 3.717785 7.083648 27.692)
-			(unlocked yes)
-			(layer "B.SilkS")
-			(effects
-				(font
-					(size 1 1)
-					(thickness 0.1)
-				)
-				(justify bottom mirror)
-			)
-		)
-		(fp_text user "CL"
-			(at -3.717785 7.083648 -27.692)
-			(unlocked yes)
-			(layer "B.SilkS")
-			(effects
-				(font
-					(size 1 1)
-					(thickness 0.1)
-				)
-				(justify bottom mirror)
-			)
-		)
-		(fp_text user "4"
-			(at -5.304981 -5.988086 -138.461)
-			(unlocked yes)
-			(layer "B.SilkS")
-			(effects
-				(font
-					(size 1 1)
-					(thickness 0.1)
-				)
-				(justify bottom mirror)
-			)
-		)
-		(fp_text user "6"
-			(at 1.914525 -7.767535 166.153)
-			(unlocked yes)
-			(layer "B.SilkS")
-			(effects
-				(font
-					(size 1 1)
-					(thickness 0.1)
-				)
-				(justify bottom mirror)
-			)
-		)
-		(fp_text user "0"
-			(at 6.583871 4.544518 55.384)
-			(unlocked yes)
-			(layer "B.SilkS")
-			(effects
-				(font
-					(size 1 1)
-					(thickness 0.1)
-				)
-				(justify bottom mirror)
-			)
-		)
-		(fp_text user "3"
-			(at -7.48013 -2.836839 -110.769)
-			(unlocked yes)
-			(layer "B.SilkS")
-			(effects
-				(font
-					(size 1 1)
-					(thickness 0.1)
-				)
-				(justify bottom mirror)
-			)
-		)
 		(fp_text user "7"
 			(at 5.304981 -5.988086 138.461)
@@
 			)
 		)
-		(fp_text user "A"
-			(at 0 8 0)
-			(unlocked yes)
-			(layer "B.SilkS")
-			(effects
-				(font
-					(size 1 1)
-					(thickness 0.1)
-				)
-				(justify bottom mirror)
-			)
-		)
-		(fp_text user "1"
-			(at -6.583871 4.544518 -55.384)
-			(unlocked yes)
-			(layer "B.SilkS")
-			(effects
-				(font
-					(size 1 1)
-					(thickness 0.1)
-				)
-				(justify bottom mirror)
-			)
-		)
-		(fp_text user "8"
-			(at 7.48013 -2.836839 110.769)
-			(unlocked yes)
-			(layer "B.SilkS")
-			(effects
-				(font
-					(size 1 1)
-					(thickness 0.1)
-				)
-				(justify bottom mirror)
-			)
-		)
-		(fp_text user "5"
-			(at -1.914525 -7.767535 -166.153)
-			(unlocked yes)
-			(layer "B.SilkS")
-			(effects
-				(font
-					(size 1 1)
-					(thickness 0.1)
-				)
-				(justify bottom mirror)
-			)
-		)
-		(fp_text user "2"
-			(at -7.941671 0.964293 -83.076)
-			(unlocked yes)
-			(layer "B.SilkS")
-			(effects
-				(font
-					(size 1 1)
-					(thickness 0.1)
-				)
-				(justify bottom mirror)
-			)
-		)
 		(fp_text user "${REFERENCE}"
 			(at 0 -2.5 0)
@@
 		(pad "1" thru_hole oval
 			(at 0 5.5 180)
-			(size 2 3)
-			(drill 0.762)
+			(size 2.25 3)
+			(drill 1.5)
 			(layers "*.Cu" "*.Mask")
 			(remove_unused_layers no)
@@
 		)
 		(pad "2" thru_hole circle
-			(at -2.555977 4.870008 152.3076923)
-			(size 2 2)
-			(drill 0.762)
+			(at -2.555977 4.870008 152.308)
+			(size 2.25 2.25)
+			(drill 1.5)
 			(layers "*.Cu" "*.Mask")
 			(remove_unused_layers no)
@@
 		)
 		(pad "3" thru_hole circle
-			(at -4.526411 3.124356 124.6153846)
-			(size 2 2)
-			(drill 0.762)
+			(at -4.526411 3.124356 124.616)
+			(size 2.25 2.25)
+			(drill 1.5)
 			(layers "*.Cu" "*.Mask")
 			(remove_unused_layers no)
@@
 		)
 		(pad "4" thru_hole circle
-			(at -5.459899 0.662952 96.92307692)
-			(size 2 2)
-			(drill 0.762)
+			(at -5.459899 0.662952 96.924)
+			(size 2.25 2.25)
+			(drill 1.5)
 			(layers "*.Cu" "*.Mask")
 			(remove_unused_layers no)
@@
 		)
 		(pad "5" thru_hole circle
-			(at -5.142589 -1.950327 69.2307692)
-			(size 2 2)
-			(drill 0.762)
+			(at -5.142589 -1.950327 69.231)
+			(size 2.25 2.25)
+			(drill 1.5)
 			(layers "*.Cu" "*.Mask")
 			(remove_unused_layers no)
@@
 		)
 		(pad "6" thru_hole circle
-			(at -3.647175 -4.116809 41.5384615)
-			(size 2 2)
-			(drill 0.762)
+			(at -3.647175 -4.116809 41.539)
+			(size 2.25 2.25)
+			(drill 1.5)
 			(layers "*.Cu" "*.Mask")
 			(remove_unused_layers no)
@@
 		)
 		(pad "7" thru_hole circle
-			(at -1.316236 -5.34018 13.8461538)
-			(size 2 2)
-			(drill 0.762)
+			(at -1.316236 -5.34018 13.847)
+			(size 2.25 2.25)
+			(drill 1.5)
 			(layers "*.Cu" "*.Mask")
 			(remove_unused_layers no)
@@
 		)
 		(pad "8" thru_hole circle
-			(at 1.316236 -5.34018 346.1538462)
-			(size 2 2)
-			(drill 0.762)
+			(at 1.316236 -5.34018 346.154)
+			(size 2.25 2.25)
+			(drill 1.5)
 			(layers "*.Cu" "*.Mask")
 			(remove_unused_layers no)
@@
 		)
 		(pad "9" thru_hole circle
-			(at 3.647175 -4.116809 318.4615385)
-			(size 2 2)
-			(drill 0.762)
+			(at 3.647175 -4.116809 318.462)
+			(size 2.25 2.25)
+			(drill 1.5)
 			(layers "*.Cu" "*.Mask")
 			(remove_unused_layers no)
@@
 		)
 		(pad "10" thru_hole circle
-			(at 5.142589 -1.950327 290.7692308)
-			(size 2 2)
-			(drill 0.762)
+			(at 5.142589 -1.950327 290.77)
+			(size 2.25 2.25)
+			(drill 1.5)
 			(layers "*.Cu" "*.Mask")
 			(remove_unused_layers no)
@@
 		)
 		(pad "11" thru_hole circle
-			(at 5.459899 0.662952 263.0769231)
-			(size 2 2)
-			(drill 0.762)
+			(at 5.459899 0.662952 263.077)
+			(size 2.25 2.25)
+			(drill 1.5)
 			(layers "*.Cu" "*.Mask")
 			(remove_unused_layers no)
@@
 		)
 		(pad "12" thru_hole circle
-			(at 4.526411 3.124356 235.3846154)
-			(size 2 2)
-			(drill 0.762)
+			(at 4.526411 3.124356 235.385)
+			(size 2.25 2.25)
+			(drill 1.5)
 			(layers "*.Cu" "*.Mask")
 			(remove_unused_layers no)
@@
 		)
 		(pad "13" thru_hole circle
-			(at 2.555977 4.870008 207.6923077)
-			(size 2 2)
-			(drill 0.762)
-			(layers "*.Cu" "*.Mask")
-			(remove_unused_layers no)
+			(at 2.555977 4.870008 207.693)
+			(size 2.25 2.25)
+			(drill 1.5)
+			(layers "*.Cu" "*.Mask")
+			(remove_unused_layers no)

Commit message: pcb changes and breakages need to fix later
Connections:
- U1 pad 1: /Comma_R -> /Comma_L
- U10 pad 1: /Cath_3 -> /Cath_8
- U11 pad 1: /Cath_4 -> /Cath_7
- U12 pad 1: /Cath_5 -> /Cath_6
- U2 pad 1: /Cath_0 -> /Cath_1
- U3 pad 1: /Cath_9 -> /Cath_2
- U4 pad 1: /Cath_8 -> /Cath_3
- U5 pad 1: /Cath_7 -> /Cath_4
- U6 pad 1: /Cath_6 -> /Cath_5
- U7 pad 1: /Comma_L -> /Comma_R
- U8 pad 1: /Cath_1 -> /Cath_0
- U9 pad 1: /Cath_2 -> /Cath_9
