File: pcb/nixie_clock/Nixie_Control.kicad_pcb (KiCad board)
At the start: 6 copper layers, 26 parts, among them U1 PCA9685BS, U10 MSD42WT1G, U11 MSD42WT1G, U12 MSD42WT1G, U13 MSD42WT1G, U2 MSD42WT1G, U3 MSD42WT1G, U4 MSD42WT1G, U5 MSD42WT1G, U6 MSD42WT1G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

Commit message: fixing some issues.
Changed lines of the file:
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@@
 			(layer "B.CrtYd")
+		)
+		(fp_text user "9"
+			(at 7.941671 0.964293 -96.924)
+			(unlocked yes)
+			(layer "B.SilkS")
+			(effects
+				(font
+					(size 1 1)
+					(thickness 0.1)
+				)
+				(justify bottom mirror)
+			)
+		)
+		(fp_text user "CR"
+			(at 3.717785 7.083648 -152.308)
+			(unlocked yes)
+			(layer "B.SilkS")
+			(effects
+				(font
+					(size 1 1)
+					(thickness 0.1)
+				)
+				(justify bottom mirror)
+			)
+		)
+		(fp_text user "2"
+			(at -7.941671 0.964293 96.924)
+			(unlocked yes)
+			(layer "B.SilkS")
+			(effects
+				(font
+					(size 1 1)
+					(thickness 0.1)
+				)
+				(justify bottom mirror)
+			)
+		)
+		(fp_text user "0"
+			(at 6.583871 4.544518 -124.616)
+			(unlocked yes)
+			(layer "B.SilkS")
+			(effects
+				(font
+					(size 1 1)
+					(thickness 0.1)
+				)
+				(justify bottom mirror)
+			)
+		)
+		(fp_text user "5"
+			(at -1.914525 -7.767535 13.847)
+			(unlocked yes)
+			(layer "B.SilkS")
+			(effects
+				(font
+					(size 1 1)
+					(thickness 0.1)
+				)
+				(justify bottom mirror)
+			)
+		)
+		(fp_text user "1"
+			(at -6.583871 4.544518 124.616)
+			(unlocked yes)
+			(layer "B.SilkS")
+			(effects
+				(font
+					(size 1 1)
+					(thickness 0.1)
+				)
+				(justify bottom mirror)
+			)
+		)
+		(fp_text user "4"
+			(at -5.304981 -5.988086 41.539)
+			(unlocked yes)
+			(layer "B.SilkS")
+			(effects
+				(font
+					(size 1 1)
+					(thickness 0.1)
+				)
+				(justify bottom mirror)
+			)
+		)
+		(fp_text user "A"
+			(at 0 8 180)
+			(unlocked yes)
+			(layer "B.SilkS")
+			(effects
+				(font
+					(size 1 1)
+					(thickness 0.1)
+				)
+				(justify bottom mirror)
+			)
+		)
+		(fp_text user "7"
+			(at 5.304981 -5.988086 -41.539)
+			(unlocked yes)
+			(layer "B.SilkS")
+			(effects
+				(font
+					(size 1 1)
+					(thickness 0.1)
+				)
+				(justify bottom mirror)
+			)
+		)
+		(fp_text user "3"
+			(at -7.48013 -2.836839 69.231)
+			(unlocked yes)
+			(layer "B.SilkS")
+			(effects
+				(font
+					(size 1 1)
+					(thickness 0.1)
+				)
+				(justify bottom mirror)
+			)
+		)
+		(fp_text user "8"
+			(at 7.48013 -2.836839 -69.231)
+			(unlocked yes)
+			(layer "B.SilkS")
+			(effects
+				(font
+					(size 1 1)
+					(thickness 0.1)
+				)
+				(justify bottom mirror)
+			)
+		)
+		(fp_text user "CL"
+			(at -3.717785 7.083648 152.308)
+			(unlocked yes)
+			(layer "B.SilkS")
+			(effects
+				(font
+					(size 1 1)
+					(thickness 0.1)
+				)
+				(justify bottom mirror)
+			)
 		)
 		(fp_text user "6"
@@
 			)
 		)
-		(fp_text user "1"
-			(at -6.583871 4.544518 124.616)
-			(unlocked yes)
-			(layer "B.SilkS")
-			(effects
-				(font
-					(size 1 1)
-					(thickness 0.1)
-				)
-				(justify bottom mirror)
-			)
-		)
-		(fp_text user "9"
-			(at 7.941671 0.964293 -96.924)
-			(unlocked yes)
-			(layer "B.SilkS")
-			(effects
-				(font
-					(size 1 1)
-					(thickness 0.1)
-				)
-				(justify bottom mirror)
-			)
-		)
-		(fp_text user "8"
-			(at 7.48013 -2.836839 -69.231)
-			(unlocked yes)
-			(layer "B.SilkS")
-			(effects
-				(font
-					(size 1 1)
-					(thickness 0.1)
-				)
-				(justify bottom mirror)
-			)
-		)
-		(fp_text user "5"
-			(at -1.914525 -7.767535 13.847)
-			(unlocked yes)
-			(layer "B.SilkS")
-			(effects
-				(font
-					(size 1 1)
-					(thickness 0.1)
-				)
-				(justify bottom mirror)
-			)
-		)
-		(fp_text user "7"
-			(at 5.304981 -5.988086 -41.539)
-			(unlocked yes)
-			(layer "B.SilkS")
-			(effects
-				(font
-					(size 1 1)
-					(thickness 0.1)
-				)
-				(justify bottom mirror)
-			)
-		)
-		(fp_text user "2"
-			(at -7.941671 0.964293 96.924)
-			(unlocked yes)
-			(layer "B.SilkS")
-			(effects
-				(font
-					(size 1 1)
-					(thickness 0.1)
-				)
-				(justify bottom mirror)
-			)
-		)
-		(fp_text user "4"
-			(at -5.304981 -5.988086 41.539)
-			(unlocked yes)
-			(layer "B.SilkS")
-			(effects
-				(font
-					(size 1 1)
-					(thickness 0.1)
-				)
-				(justify bottom mirror)
-			)
-		)
-		(fp_text user "CR"
-			(at 3.717785 7.083648 -152.308)
-			(unlocked yes)
-			(layer "B.SilkS")
-			(effects
-				(font
-					(size 1 1)
-					(thickness 0.1)
-				)
-				(justify bottom mirror)
-			)
-		)
-		(fp_text user "A"
-			(at 0 8 180)
-			(unlocked yes)
-			(layer "B.SilkS")
-			(effects
-				(font
-					(size 1 1)
-					(thickness 0.1)
-				)
-				(justify bottom mirror)
-			)
-		)
-		(fp_text user "0"
-			(at 6.583871 4.544518 -124.616)
-			(unlocked yes)
-			(layer "B.SilkS")
-			(effects
-				(font
-					(size 1 1)
-					(thickness 0.1)
-				)
-				(justify bottom mirror)
-			)
-		)
-		(fp_text user "3"
-			(at -7.48013 -2.836839 69.231)
-			(unlocked yes)
-			(layer "B.SilkS")
-			(effects
-				(font
-					(size 1 1)
-					(thickness 0.1)
-				)
-				(justify bottom mirror)
-			)
-		)
-		(fp_text user "CL"
-			(at -3.717785 7.083648 152.308)
-			(unlocked yes)
-			(layer "B.SilkS")
-			(effects
-				(font
-					(size 1 1)
-					(thickness 0.1)
-				)
-				(justify bottom mirror)
-			)
-		)
 		(fp_text user "${REFERENCE}"
 			(at 0 -2.5 180)
@@
 		(pad "1" thru_hole oval
 			(at 0 5.5)
-			(size 2 3)
-			(drill 0.762)
+			(size 2.25 3)
+			(drill 1.5)
 			(layers "*.Cu" "*.Mask")
 			(remove_unused_layers no)
@@
 		)
 		(pad "2" thru_hole circle
-			(at -2.555977 4.870008 332.3076923)
-			(size 2 2)
-			(drill 0.762)
+			(at -2.555977 4.870008 332.308)
+			(size 2.25 2.25)
+			(drill 1.5)
 			(layers "*.Cu" "*.Mask")
 			(remove_unused_layers no)
@@
 		)
 		(pad "3" thru_hole circle
-			(at -4.526411 3.124356 304.6153846)
-			(size 2 2)
-			(drill 0.762)
+			(at -4.526411 3.124356 304.616)
+			(size 2.25 2.25)
+			(drill 1.5)
 			(layers "*.Cu" "*.Mask")
 			(remove_unused_layers no)
@@
 		)
 		(pad "4" thru_hole circle
-			(at -5.459899 0.662952 276.9230769)
-			(size 2 2)
-			(drill 0.762)
+			(at -5.459899 0.662952 276.924)
+			(size 2.25 2.25)
+			(drill 1.5)
 			(layers "*.Cu" "*.Mask")
 			(remove_unused_layers no)
@@
 		)
 		(pad "5" thru_hole circle
-			(at -5.142589 -1.950327 249.2307692)
-			(size 2 2)
-			(drill 0.762)
+			(at -5.142589 -1.950327 249.231)
+			(size 2.25 2.25)
+			(drill 1.5)
 			(layers "*.Cu" "*.Mask")
 			(remove_unused_layers no)
@@
 		)
 		(pad "6" thru_hole circle
-			(at -3.647175 -4.116809 221.5384615)
-			(size 2 2)
-			(drill 0.762)
+			(at -3.647175 -4.116809 221.539)
+			(size 2.25 2.25)
+			(drill 1.5)
 			(layers "*.Cu" "*.Mask")
 			(remove_unused_layers no)
@@
 		)
 		(pad "7" thru_hole circle
-			(at -1.316236 -5.34018 193.8461538)
-			(size 2 2)
-			(drill 0.762)
+			(at -1.316236 -5.34018 193.847)
+			(size 2.25 2.25)
+			(drill 1.5)
 			(layers "*.Cu" "*.Mask")
 			(remove_unused_layers no)
@@
 		)
 		(pad "8" thru_hole circle
-			(at 1.316236 -5.34018 166.1538462)
-			(size 2 2)
-			(drill 0.762)
+			(at 1.316236 -5.34018 166.154)
+			(size 2.25 2.25)
+			(drill 1.5)
 			(layers "*.Cu" "*.Mask")
 			(remove_unused_layers no)
@@
 		)
 		(pad "9" thru_hole circle
-			(at 3.647175 -4.116809 138.4615385)
-			(size 2 2)
-			(drill 0.762)
+			(at 3.647175 -4.116809 138.462)
+			(size 2.25 2.25)
+			(drill 1.5)
 			(layers "*.Cu" "*.Mask")
 			(remove_unused_layers no)
@@
 		)
 		(pad "10" thru_hole circle
-			(at 5.142589 -1.950327 110.7692308)
-			(size 2 2)
-			(drill 0.762)
+			(at 5.142589 -1.950327 110.77)
+			(size 2.25 2.25)
+			(drill 1.5)
 			(layers "*.Cu" "*.Mask")
 			(remove_unused_layers no)
@@
 		)
 		(pad "11" thru_hole circle
-			(at 5.459899 0.662952 83.0769231)
-			(size 2 2)
-			(drill 0.762)
+			(at 5.459899 0.662952 83.077)
+			(size 2.25 2.25)
+			(drill 1.5)
 			(layers "*.Cu" "*.Mask")
 			(remove_unused_layers no)
@@
 		)
 		(pad "12" thru_hole circle
-			(at 4.526411 3.124356 55.3846154)
-			(size 2 2)
-			(drill 0.762)
+			(at 4.526411 3.124356 55.385)
+			(size 2.25 2.25)
+			(drill 1.5)
 			(layers "*.Cu" "*.Mask")
 			(remove_unused_layers no)
@@
 		)
 		(pad "13" thru_hole circle
-			(at 2.555977 4.870008 27.6923077)
-			(size 2 2)
-			(drill 0.762)
+			(at 2.555977 4.870008 27.693)
+			(size 2.25 2.25)
+			(drill 1.5)
 			(layers "*.Cu" "*.Mask")
 			(remove_unused_layers no)
@@
 			(pintype "output")
 		)
+		(zone
+			(net 0)
+			(net_name "")
+			(layers "*.Cu")
+			(hatch edge 0.5)
+			(connect_pads
+				(clearance 0)
+			)
+			(min_thickness 0.25)
+			(filled_areas_thickness no)
+			(keepout
+				(tracks not_allowed)
+				(vias not_allowed)
+				(pads not_allowed)
+				(copperpour not_allowed)
+				(footprints allowed)
+			)
+			(fill
+				(thermal_gap 0.5)
+				(thermal_bridge_width 0.5)
+			)
+			(polygon
+				(pts
+					(xy 158.7275 85.7) (xy 158.2275 83.7) (xy 158.2275 81.7) (xy 159.2275 80.2) (xy 161.2275 79.2)
+					(xy 163.2275 79.2) (xy 165.2275 80.2) (xy 166.2275 82.2) (xy 166.2275 83.7) (xy 165.7275 85.2)
+					(xy 164.2275 86.7) (xy 162.2275 86.7) (xy 160.2275 86.7)
+				)
+			)
+		)
 	)

Commit message: added grounding
Routing:
- net /Nixie_Block2/Cath_6: track 34.6 -> 35.2 mm
Changed lines of the file:
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@@
 	)
 	(segment
-		(start 170.2 87.584314)
-		(end 170.2 76.05)
+		(start 165.808579 91.975735)
+		(end 170.8 86.984314)
 		(width 0.2)
 		(layer "B.Cu")
@@
 	)
 	(segment
-		(start 170.2 76.05)
-		(end 168.7 74.55)
+		(start 165.808579 96.908579)
+		(end 165.808579 91.975735)
 		(width 0.2)
 		(layer "B.Cu")
@@
 	)
 	(segment
-		(start 165.808579 91.975735)
-		(end 170.2 87.584314)
+		(start 170.8 86.984314)
+		(end 170.8 76.65)
 		(width 0.2)
 		(layer "B.Cu")
@@
 	)
 	(segment
-		(start 165.808579 91.975735)
-		(end 165.808579 96.908579)
+		(start 170.8 76.65)
+		(end 168.7 74.55)
 		(width 0.2)
 		(layer "B.Cu")
@@
 	)
 	(segment
-		(start 169.15 85.766745)
-		(end 169.15 78.3)
+		(start 165.191422 98.091422)
+		(end 165.191422 90.908578)
 		(width 0.2)
 		(layer "B.Cu")
@@
 	)
 	(segment
-		(start 165.191422 89.725323)
-		(end 165.191422 98.091422)
+		(start 165.191422 90.908578)
+		(end 169.8 86.3)
 		(width 0.2)
 		(layer "B.Cu")
@@
 	)
 	(segment
-		(start 165.191422 89.725323)
-		(end 169.15 85.766745)
+		(start 169.8 78.95)
+		(end 166 75.15)
 		(width 0.2)
 		(layer "B.Cu")
@@
 	)
 	(segment
-		(start 169.15 78.3)
-		(end 166 75.15)
+		(start 169.8 86.3)
+		(end 169.8 78.95)
 		(width 0.2)
 		(layer "B.Cu")

Commit message: pcb changes and breakages need to fix later
Connections:
- net +5V renamed +3V3
- net /Ext_Clk renamed /Out_En
- U10 pad 1: /Nixie_Block2/Cath_2 -> /Nixie_Block2/Cath_9
- U11 pad 1: /Nixie_Block2/Cath_3 -> /Nixie_Block2/Cath_8
- U12 pad 1: /Nixie_Block2/Cath_4 -> /Nixie_Block2/Cath_7
- U13 pad 1: /Nixie_Block2/Cath_5 -> /Nixie_Block2/Cath_6
- U2 pad 1: /Nixie_Block2/Comma_R -> /Nixie_Block2/Comma_L
- U3 pad 1: /Nixie_Block2/Cath_0 -> /Nixie_Block2/Cath_1
- U4 pad 1: /Nixie_Block2/Cath_9 -> /Nixie_Block2/Cath_2
- U5 pad 1: /Nixie_Block2/Cath_8 -> /Nixie_Block2/Cath_3
- U6 pad 1: /Nixie_Block2/Cath_7 -> /Nixie_Block2/Cath_4
- U7 pad 1: /Nixie_Block2/Cath_6 -> /Nixie_Block2/Cath_5
- U8 pad 1: /Nixie_Block2/Comma_L -> /Nixie_Block2/Comma_R
- U9 pad 1: /Nixie_Block2/Cath_1 -> /Nixie_Block2/Cath_0
