File: pcb/nixie_clock/nixie_clock.kicad_sch (KiCad schematic)
At the start: 1 part, among them J1 Conn_01x06_Pin

Commit message: final commits before sending to jlc
Parts:
- added H1, H2, H3, H4: MountingHole_Pad, MountingHole:MountingHole_2.7mm_M2.5_DIN965_Pad, symbol Mechanical:MountingHole_Pad
- J1: now fitted; now left out of the parts list
Connections:
- net GND: now also H1.1, H2.1, H3.1, H4.1
Other:
- sheet Nixie_Control ports: added Out_En; removed Ext_Clk
- sheet Nixie_Control1 ports: added Out_En; removed Ext_Clk
- sheet Nixie_Control2 ports: added Out_En; removed Ext_Clk
- sheet Nixie_Control3 ports: added Out_En; removed Ext_Clk
- sheet Nixie_Control4 ports: added Out_En; removed Ext_Clk
